Commit message: refactor code, add amr_lidars, update environment variables, update scan safety

File: amr_simulation/urdf/control/gazebo_sim_ros2_control.urdf.xacro (robot description, xacro)
@@ -1,9 +1,9 @@
 <?xml version="1.0" ?>
 <robot xmlns:xacro="http://wiki.ros.org/xacro">
-    <xacro:macro name="load_gazebo_sim_ros2_control_plugin" params="robot_name use_gazebo">
+    <xacro:macro name="load_gazebo_sim_ros2_control_plugin" params="robot_name use_gazebo controllers_file">
         <xacro:if value="${use_gazebo}">
             <gazebo>
                 <plugin filename="gz_ros2_control-system" name="gz_ros2_control::GazeboSimROS2ControlPlugin">
-                    <parameters>$(find amr_simulation)/config/${robot_name}/ros2_controllers.yaml</parameters>
+                    <parameters>${controllers_file}</parameters>
                     <ros>
                         <remapping>/controller_manager/robot_description:=/robot_description</remapping>

File: amr_simulation/urdf/robots/mecanum_drive.urdf.xacro (robot description, xacro)
@@ -5,4 +5,5 @@
     <xacro:arg name="prefix" default=""/>
     <xacro:arg name="use_gazebo" default="false"/>
+    <xacro:arg name="controllers_file" default="$(optenv CONFIG_FOLDER /var/amr/config)/mecanum/ros2_controllers.yaml"/>
     <!-- Changed rosmaster_x3_base to mecanum_base -->
     <xacro:include filename="$(find amr_simulation)/urdf/mech/mecanum_base.urdf.xacro"/>
@@ -63,4 +64,5 @@
     <xacro:load_gazebo_sim_ros2_control_plugin
       robot_name="$(arg robot_name)"
+      controllers_file="$(arg controllers_file)"
       use_gazebo="$(arg use_gazebo)"/>
     <xacro:include filename="$(find amr_simulation)/urdf/control/mecanum_ros2_control.urdf.xacro" />
