Commit message: chore: fix elay time to run gazebo simulation, commen velocity plugin which as a result of stafing motion

File: amr_simulation/urdf/control/velocity_control_plugin.urdf.xacro (robot description, xacro)
@@ -7,5 +7,5 @@
                     filename="gz-sim-velocity-control-system"
                     name="gz::sim::systems::VelocityControl">
-                    <topic>mecanum_drive_controller/cmd_vel</topic>
+                    <topic>cmd_vel</topic>
                     <initial_linear>0 0 0</initial_linear>
                     <initial_angular>0 0 0</initial_angular>

File: amr_simulation/urdf/mech/mecanum_wheel.urdf.xacro (robot description, xacro)
@@ -1,4 +1,5 @@
 <?xml version="1.0"?>
-<robot xmlns:xacro="http://www.ros.org/wiki/xacro">
+<robot xmlns:xacro="http://www.ros.org/wiki/xacro"
+       xmlns:ignition="http://gazebosim.org/schema">
   <xacro:property name="wheel_radius" value="0.0325" />
   <xacro:property name="wheel_separation" value="0.169" />
@@ -40,12 +41,15 @@
     </joint>
     <gazebo reference="${prefix}${side}_wheel_link">
-      <surface>
-        <friction>
-          <ode>
+      <collision>
+        <surface>
+          <friction>
+            <ode>
               <mu>1.0</mu>
               <mu2>0.0</mu2>
-          </ode>
-        </friction>
-      </surface>
+              <fdir1 ignition:expressed_in="${prefix}base_footprint">1 ${-x_reflect*y_reflect} 0</fdir1>
+            </ode>
+          </friction>
+        </surface>
+      </collision>
       <visual>
           <material>

File: amr_simulation/urdf/robots/mecanum_drive.urdf.xacro (robot description, xacro)
@@ -34,9 +34,9 @@
       x_reflect="-1"
       y_reflect="-1"/>
-    <xacro:rgbd_camera
+    <!-- <xacro:rgbd_camera
       prefix="$(arg prefix)"
       camera_name="cam_1"
       xyz_offset="0.105 0 0.05"
-      rpy_offset="0 -0.50 0"/>
+      rpy_offset="0 -0.50 0"/> -->
     <xacro:lidar_sensor
       prefix="$(arg prefix)"
@@ -59,5 +59,5 @@
     -->
     <xacro:include filename="$(find amr_simulation)/urdf/control/velocity_control_plugin.urdf.xacro" />
-    <xacro:load_velocity_control_plugin use_gazebo="$(arg use_gazebo)"/>
+    <!-- <xacro:load_velocity_control_plugin use_gazebo="$(arg use_gazebo)"/> -->
     <xacro:include filename="$(find amr_simulation)/urdf/control/gazebo_sim_ros2_control.urdf.xacro" />
     <xacro:load_gazebo_sim_ros2_control_plugin
